Commit message: Updated readme with first footsteps

File: unitree_g1/g1.urdf (robot description, URDF)
Before this commit: robot converted_robot, 89 links, 88 joints
Links:
- removed link left_hand_index_0_joint_jointbody
- removed link left_hand_index_0_link
- removed link left_hand_index_1_joint_jointbody
- removed link left_hand_index_1_link
- removed link left_hand_middle_0_joint_jointbody
- removed link left_hand_middle_0_link
- removed link left_hand_middle_1_joint_jointbody
- removed link left_hand_middle_1_link
- removed link left_hand_thumb_0_joint_jointbody
- removed link left_hand_thumb_0_link
- removed link left_hand_thumb_1_joint_jointbody
- removed link left_hand_thumb_1_link
- removed link left_hand_thumb_2_joint_jointbody
- removed link left_hand_thumb_2_link
- removed link right_hand_index_0_joint_jointbody
- removed link right_hand_index_0_link
- removed link right_hand_index_1_joint_jointbody
- removed link right_hand_index_1_link
- removed link right_hand_middle_0_joint_jointbody
- removed link right_hand_middle_0_link
- removed link right_hand_middle_1_joint_jointbody
- removed link right_hand_middle_1_link
- removed link right_hand_thumb_0_joint_jointbody
- removed link right_hand_thumb_0_link
- removed link right_hand_thumb_1_joint_jointbody
- removed link right_hand_thumb_1_link
- removed link right_hand_thumb_2_joint_jointbody
- removed link right_hand_thumb_2_link
- link left_ankle_pitch_link: geometry visual mesh filename=meshes/converted_left_ankle_pitch_link_b2b2b2ff.obj
- link left_ankle_roll_link: geometry visual mesh filename=meshes/converted_left_ankle_roll_link_333333ff.obj
- link left_elbow_link: geometry visual mesh filename=meshes/converted_left_elbow_link_b2b2b2ff.obj
- link left_hip_pitch_link: geometry visual mesh filename=meshes/converted_left_hip_pitch_link_333333ff.obj
- link left_hip_roll_link: geometry visual mesh filename=meshes/converted_left_hip_roll_link_b2b2b2ff.obj
- link left_hip_yaw_link: geometry visual mesh filename=meshes/converted_left_hip_yaw_link_b2b2b2ff.obj
- link left_knee_link: geometry visual mesh filename=meshes/converted_left_knee_link_b2b2b2ff.obj
- link left_shoulder_pitch_link: geometry visual mesh filename=meshes/converted_left_shoulder_pitch_link_b2b2b2ff.obj
- link left_shoulder_roll_link: geometry visual mesh filename=meshes/converted_left_shoulder_roll_link_b2b2b2ff.obj
- link left_shoulder_yaw_link: geometry visual mesh filename=meshes/converted_left_shoulder_yaw_link_b2b2b2ff.obj
- link left_wrist_pitch_link: geometry visual mesh filename=meshes/converted_left_wrist_pitch_link_b2b2b2ff.obj
- link left_wrist_roll_link: geometry visual mesh filename=meshes/converted_left_wrist_roll_link_b2b2b2ff.obj
- link left_wrist_yaw_link: mass 0.457415 -> 0.254576; geometry visual mesh filename=meshes/converted_left_rubber_hand_b2b2b2ff.obj; visual mesh filename=meshes/converted_left_wrist_yaw_link_b2b2b2ff.obj
- link pelvis: geometry visual mesh filename=meshes/converted_pelvis_333333ff.obj; visual mesh filename=meshes/converted_pelvis_contour_link_b2b2b2ff.obj
- link right_ankle_pitch_link: geometry visual mesh filename=meshes/converted_right_ankle_pitch_link_b2b2b2ff.obj
- link right_ankle_roll_link: geometry visual mesh filename=meshes/converted_right_ankle_roll_link_333333ff.obj
- link right_elbow_link: geometry visual mesh filename=meshes/converted_right_elbow_link_b2b2b2ff.obj
- link right_hip_pitch_link: geometry visual mesh filename=meshes/converted_right_hip_pitch_link_333333ff.obj
- link right_hip_roll_link: geometry visual mesh filename=meshes/converted_right_hip_roll_link_b2b2b2ff.obj
- link right_hip_yaw_link: geometry visual mesh filename=meshes/converted_right_hip_yaw_link_b2b2b2ff.obj
- link right_knee_link: geometry visual mesh filename=meshes/converted_right_knee_link_b2b2b2ff.obj
- link right_shoulder_pitch_link: geometry visual mesh filename=meshes/converted_right_shoulder_pitch_link_b2b2b2ff.obj
- link right_shoulder_roll_link: geometry visual mesh filename=meshes/converted_right_shoulder_roll_link_b2b2b2ff.obj
- link right_shoulder_yaw_link: geometry visual mesh filename=meshes/converted_right_shoulder_yaw_link_b2b2b2ff.obj
- link right_wrist_pitch_link: geometry visual mesh filename=meshes/converted_right_wrist_pitch_link_b2b2b2ff.obj
- link right_wrist_roll_link: geometry visual mesh filename=meshes/converted_right_wrist_roll_link_b2b2b2ff.obj
- link right_wrist_yaw_link: mass 0.457415 -> 0.254576; geometry visual mesh filename=meshes/converted_right_rubber_hand_b2b2b2ff.obj; visual mesh filename=meshes/converted_right_wrist_yaw_link_b2b2b2ff.obj
- link torso_link: geometry visual mesh filename=meshes/converted_head_link_333333ff.obj; visual mesh filename=meshes/converted_logo_link_333333ff.obj
- link waist_roll_link: geometry visual mesh filename=meshes/converted_waist_roll_link_b2b2b2ff.obj
- link waist_yaw_link: geometry visual mesh filename=meshes/converted_waist_yaw_link_b2b2b2ff.obj
Joints:
- removed joint left_hand_index_0_joint
- removed joint left_hand_index_0_joint_offset
- removed joint left_hand_index_1_joint
- removed joint left_hand_index_1_joint_offset
- removed joint left_hand_middle_0_joint
- removed joint left_hand_middle_0_joint_offset
- removed joint left_hand_middle_1_joint
- removed joint left_hand_middle_1_joint_offset
- removed joint left_hand_thumb_0_joint
- removed joint left_hand_thumb_0_joint_offset
- removed joint left_hand_thumb_1_joint
- removed joint left_hand_thumb_1_joint_offset
- removed joint left_hand_thumb_2_joint
- removed joint left_hand_thumb_2_joint_offset
- removed joint right_hand_index_0_joint
- removed joint right_hand_index_0_joint_offset
- removed joint right_hand_index_1_joint
- removed joint right_hand_index_1_joint_offset
- removed joint right_hand_middle_0_joint
- removed joint right_hand_middle_0_joint_offset
- removed joint right_hand_middle_1_joint
- removed joint right_hand_middle_1_joint_offset
- removed joint right_hand_thumb_0_joint
- removed joint right_hand_thumb_0_joint_offset
- removed joint right_hand_thumb_1_joint
- removed joint right_hand_thumb_1_joint_offset
- removed joint right_hand_thumb_2_joint
- removed joint right_hand_thumb_2_joint_offset

File: unitree_g1/g1_with_hands.urdf (robot description, URDF)
Before this commit: robot converted_robot, 89 links, 88 joints
Links:
- removed link floating_base_joint_jointbody
- removed link world
Joints:
- removed joint floating_base_joint
- removed joint floating_base_joint_offset
